File: DFPs.kicad_sch (KiCad schematic)
At the start: 18 parts

Commit message: good first pass
Other:
- company: (none) -> https://pips.engineering
- title: (none) -> Downstream-facing ports
Changed lines of the file:
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@@
 	(generator_version "9.0")
 	(paper "A4")
+	(title_block
+		(title "Downstream-facing ports")
+		(date "2025-12-10")
+		(rev "R1")
+		(company "https://pips.engineering")
+	)
 	(junction
 		(at 163.83 113.03)
@@
 		)
 	)
+	(table
+		(column_count 2)
+		(border
+			(external yes)
+			(header yes)
+			(stroke
+				(width 0)
+				(type solid)
+			)
+		)
+		(separators
+			(rows yes)
+			(cols yes)
+			(stroke
+				(width 0)
+				(type solid)
+			)
+		)
+		(column_widths 11.43 10.16)
+		(row_heights 2.54 2.54 2.54 2.54)
+		(cells
+			(table_cell "CC value"
+				(exclude_from_sim no)
+				(at 107.95 173.99 0)
+				(size 11.43 2.54)
+				(margins 0.9525 0.9525 0.9525 0.9525)
+				(span 1 1)
+				(fill
+					(type none)
+				)
+				(effects
+					(font
+						(size 1.27 1.27)
+						(thickness 0.254)
+						(bold yes)
+					)
+					(justify left top)
+				)
+			)
+			(table_cell "Current"
+				(exclude_from_sim no)
+				(at 119.38 173.99 0)
+				(size 10.16 2.54)
+				(margins 0.9525 0.9525 0.9525 0.9525)
+				(span 1 1)
+				(fill
+					(type none)
+				)
+				(effects
+					(font
+						(size 1.27 1.27)
+						(thickness 0.254)
+						(bold yes)
+					)
+					(justify left top)
+				)
+			)
+			(table_cell "56kΩ"
+				(exclude_from_sim no)
+				(at 107.95 176.53 0)
+				(size 11.43 2.54)
+				(margins 0.9525 0.9525 0.9525 0.9525)
+				(span 1 1)
+				(fill
+					(type none)
+				)
+				(effects
+					(font
+						(size 1.27 1.27)
+					)
+					(justify left top)
+				)
+			)
+			(table_cell "500mA"
+				(exclude_from_sim no)
+				(at 119.38 176.53 0)
+				(size 10.16 2.54)
+				(margins 0.9525 0.9525 0.9525 0.9525)
+				(span 1 1)
+				(fill
+					(type none)
+				)
+				(effects
+					(font
+						(size 1.27 1.27)
+					)
+					(justify left top)
+				)
+			)
+			(table_cell "22kΩ"
+				(exclude_from_sim no)
+				(at 107.95 179.07 0)
+				(size 11.43 2.54)
+				(margins 0.9525 0.9525 0.9525 0.9525)
+				(span 1 1)
+				(fill
+					(type none)
+				)
+				(effects
+					(font
+						(size 1.27 1.27)
+					)
+					(justify left top)
+				)
+			)
+			(table_cell "1.5A"
+				(exclude_from_sim no)
+				(at 119.38 179.07 0)
+				(size 10.16 2.54)
+				(margins 0.9525 0.9525 0.9525 0.9525)
+				(span 1 1)
+				(fill
+					(type none)
+				)
+				(effects
+					(font
+						(size 1.27 1.27)
+					)
+					(justify left top)
+				)
+			)
+			(table_cell "10kΩ"
+				(exclude_from_sim no)
+				(at 107.95 181.61 0)
+				(size 11.43 2.54)
+				(margins 0.9525 0.9525 0.9525 0.9525)
+				(span 1 1)
+				(fill
+					(type none)
+				)
+				(effects
+					(font
+						(size 1.27 1.27)
+					)
+					(justify left top)
+				)
+			)
+			(table_cell "3A"
+				(exclude_from_sim no)
+				(at 119.38 181.61 0)
+				(size 10.16 2.54)
+				(margins 0.9525 0.9525 0.9525 0.9525)
+				(span 1 1)
+				(fill
+					(type none)
+				)
+				(effects
+					(font
+						(size 1.27 1.27)
+					)
+					(justify left top)
+				)
+			)
+		)
+	)
 	(hierarchical_label "DFP_VBUS"
 		(shape bidirectional)
-		(at 220.98 73.66 0)
+		(at 220.98 73.66 90)
 		(effects
 			(font
@@
 	(hierarchical_label "DFP_VBUS"
 		(shape bidirectional)
-		(at 262.89 73.66 0)
+		(at 262.89 73.66 90)
 		(effects
 			(font
@@
 	(hierarchical_label "DFP_VBUS"
 		(shape bidirectional)
-		(at 53.34 73.66 0)
+		(at 53.34 73.66 90)
 		(effects
 			(font
@@
 	(hierarchical_label "DFP_VBUS"
 		(shape bidirectional)
-		(at 179.07 73.66 0)
+		(at 179.07 73.66 90)
 		(effects
 			(font
@@
 	(hierarchical_label "DFP_VBUS"
 		(shape bidirectional)
-		(at 95.25 73.66 0)
+		(at 95.25 73.66 90)
 		(effects
 			(font
@@
 	(hierarchical_label "DFP_VBUS"
 		(shape bidirectional)
-		(at 137.16 73.66 0)
-		(effects
-			(font
+		(at 137.16 73.66 90)
+		(effects
+			(font

Commit message: more work on USB hubs
Parts:
- renumbered R3 to R19, R4 to R20, R5 to R21, R6 to R22, R7 to R23, R8 to R24, R9 to R25, R10 to R26, R11 to R27, R12 to R28, R13 to R29, R14 to R30
Changed lines of the file:
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@@
 			(table_cell "CC value"
 				(exclude_from_sim no)
-				(at 107.95 173.99 0)
+				(at 26.67 41.91 0)
 				(size 11.43 2.54)
 				(margins 0.9525 0.9525 0.9525 0.9525)
@@
 			(table_cell "Current"
 				(exclude_from_sim no)
-				(at 119.38 173.99 0)
+				(at 38.1 41.91 0)
 				(size 10.16 2.54)
 				(margins 0.9525 0.9525 0.9525 0.9525)
@@
 			(table_cell "56kΩ"
 				(exclude_from_sim no)
-				(at 107.95 176.53 0)
+				(at 26.67 44.45 0)
 				(size 11.43 2.54)
 				(margins 0.9525 0.9525 0.9525 0.9525)
@@
 			(table_cell "500mA"
 				(exclude_from_sim no)
-				(at 119.38 176.53 0)
+				(at 38.1 44.45 0)
 				(size 10.16 2.54)
 				(margins 0.9525 0.9525 0.9525 0.9525)
@@
 			(table_cell "22kΩ"
 				(exclude_from_sim no)
-				(at 107.95 179.07 0)
+				(at 26.67 46.99 0)
 				(size 11.43 2.54)
 				(margins 0.9525 0.9525 0.9525 0.9525)
@@
 			(table_cell "1.5A"
 				(exclude_from_sim no)
-				(at 119.38 179.07 0)
+				(at 38.1 46.99 0)
 				(size 10.16 2.54)
 				(margins 0.9525 0.9525 0.9525 0.9525)
@@
 			(table_cell "10kΩ"
 				(exclude_from_sim no)
-				(at 107.95 181.61 0)
+				(at 26.67 49.53 0)
 				(size 11.43 2.54)
 				(margins 0.9525 0.9525 0.9525 0.9525)
@@
 			(table_cell "3A"
 				(exclude_from_sim no)
-				(at 119.38 181.61 0)
+				(at 38.1 49.53 0)
 				(size 10.16 2.54)
 				(margins 0.9525 0.9525 0.9525 0.9525)
@@
 		(on_board yes)
 		(dnp no)
-		(property "Reference" "R11"
+		(property "Reference" "R27"
 			(at 221.996 76.454 0)
 			(effects
@@
 			(project "Multiport USB-C 2.0 hub"
 				(path "/36dda7fd-e284-4ee0-b9cb-842fdde3c54e/842043d2-bca2-4e2b-b4fa-303380c6ca60"
-					(reference "R11")
+					(reference "R27")
 					(unit 1)
 				)
@@
 		(on_board yes)
 		(dnp no)
-		(property "Reference" "R3"
+		(property "Reference" "R19"
 			(at 54.356 76.454 0)
 			(effects
@@
 			(project ""
 				(path "/36dda7fd-e284-4ee0-b9cb-842fdde3c54e/842043d2-bca2-4e2b-b4fa-303380c6ca60"
-					(reference "R3")
+					(reference "R19")
 					(unit 1)
 				)
@@
 		(on_board yes)
 		(dnp no)
-		(property "Reference" "R8"
+		(property "Reference" "R24"
 			(at 145.796 76.454 0)
 			(effects
@@
 			(project "Multiport USB-C 2.0 hub"
 				(path "/36dda7fd-e284-4ee0-b9cb-842fdde3c54e/842043d2-bca2-4e2b-b4fa-303380c6ca60"
-					(reference "R8")
+					(reference "R24")
 					(unit 1)
 				)
@@
 		(on_board yes)
 		(dnp no)
-		(property "Reference" "R6"
+		(property "Reference" "R22"
 			(at 103.886 76.454 0)
 			(effects
@@
 			(project "Multiport USB-C 2.0 hub"
 				(path "/36dda7fd-e284-4ee0-b9cb-842fdde3c54e/842043d2-bca2-4e2b-b4fa-303380c6ca60"
-					(reference "R6")
+					(reference "R22")
 					(unit 1)
 				)
@@
 		(dnp no)
 		(fields_autoplaced yes)
-		(property "Reference" "#PWR06"
+		(property "Reference" "#PWR026"
 			(at 38.1 119.38 0)
 			(effects
@@
 			(project "Multiport USB-C 2.0 hub"
 				(path "/36dda7fd-e284-4ee0-b9cb-842fdde3c54e/842043d2-bca2-4e2b-b4fa-303380c6ca60"
-					(reference "#PWR06")
+					(reference "#PWR026")
 					(unit 1)
 				)
@@
 		(dnp no)
 		(fields_autoplaced yes)
-		(property "Reference" "#PWR010"
+		(property "Reference" "#PWR031"
 			(at 247.65 119.38 0)
 			(effects
@@
 			(project "Multiport USB-C 2.0 hub"
 				(path "/36dda7fd-e284-4ee0-b9cb-842fdde3c54e/842043d2-bca2-4e2b-b4fa-303380c6ca60"
-					(reference "#PWR010")
+					(reference "#PWR031")
 					(unit 1)
 				)
@@
 		(dnp no)
 		(fields_autoplaced yes)
-		(property "Reference" "#PWR09"
+		(property "Reference" "#PWR030"
 			(at 205.74 119.38 0)
 			(effects
@@
 			(project "Multiport USB-C 2.0 hub"
 				(path "/36dda7fd-e284-4ee0-b9cb-842fdde3c54e/842043d2-bca2-4e2b-b4fa-303380c6ca60"
-					(reference "#PWR09")
+					(reference "#PWR030")
 					(unit 1)
 				)
@@
 		(on_board yes)
 		(dnp no)
-		(property "Reference" "R7"
+		(property "Reference" "R23"
 			(at 138.176 76.454 0)
 			(effects
@@
 			(project "Multiport USB-C 2.0 hub"
 				(path "/36dda7fd-e284-4ee0-b9cb-842fdde3c54e/842043d2-bca2-4e2b-b4fa-303380c6ca60"
-					(reference "R7")
+					(reference "R23")
 					(unit 1)
 				)
@@
 		(on_board yes)
 		(dnp no)
-		(property "Reference" "R13"
+		(property "Reference" "R29"
 			(at 263.906 76.454 0)
 			(effects
@@
 			(project "Multiport USB-C 2.0 hub"
 				(path "/36dda7fd-e284-4ee0-b9cb-842fdde3c54e/842043d2-bca2-4e2b-b4fa-303380c6ca60"
-					(reference "R13")
+					(reference "R29")
 					(unit 1)
 				)
@@
 		(on_board yes)
 		(dnp no)
-		(property "Reference" "R12"
+		(property "Reference" "R28"
 			(at 229.616 76.454 0)
 			(effects
@@
 			(project "Multiport USB-C 2.0 hub"
 				(path "/36dda7fd-e284-4ee0-b9cb-842fdde3c54e/842043d2-bca2-4e2b-b4fa-303380c6ca60"
-					(reference "R12")
+					(reference "R28")
 					(unit 1)
 				)
@@
 		(on_board yes)
 		(dnp no)
-		(property "Reference" "R4"
+		(property "Reference" "R20"
 			(at 61.976 76.454 0)
 			(effects
@@
 			(project "Multiport USB-C 2.0 hub"
 				(path "/36dda7fd-e284-4ee0-b9cb-842fdde3c54e/842043d2-bca2-4e2b-b4fa-303380c6ca60"
-					(reference "R4")
+					(reference "R20")
 					(unit 1)
 				)
@@
 		(on_board yes)
 		(dnp no)
-		(property "Reference" "R14"
+		(property "Reference" "R30"
 			(at 271.526 76.454 0)
 			(effects
@@
 			(project "Multiport USB-C 2.0 hub"
 				(path "/36dda7fd-e284-4ee0-b9cb-842fdde3c54e/842043d2-bca2-4e2b-b4fa-303380c6ca60"
-					(reference "R14")
+					(reference "R30")
 					(unit 1)
 				)
@@
 		(dnp no)
 		(fields_autoplaced yes)
-		(property "Reference" "#PWR08"
+		(property "Reference" "#PWR029"
 			(at 163.83 119.38 0)
 			(effects
@@
 			(project "Multiport USB-C 2.0 hub"
 				(path "/36dda7fd-e284-4ee0-b9cb-842fdde3c54e/842043d2-bca2-4e2b-b4fa-303380c6ca60"
-					(reference "#PWR08")
+					(reference "#PWR029")
 					(unit 1)
 				)
@@
 		(dnp no)
 		(fields_autoplaced yes)
-		(property "Reference" "#PWR05"
+		(property "Reference" "#PWR027"
 			(at 80.01 119.38 0)
 			(effects
@@
 			(project "Multiport USB-C 2.0 hub"
 				(path "/36dda7fd-e284-4ee0-b9cb-842fdde3c54e/842043d2-bca2-4e2b-b4fa-303380c6ca60"
-					(reference "#PWR05")
+					(reference "#PWR027")
 					(unit 1)
 				)
@@
 		(on_board yes)
 		(dnp no)
-		(property "Reference" "R10"
+		(property "Reference" "R26"
 			(at 187.706 76.454 0)
 			(effects
@@
 			(project "Multiport USB-C 2.0 hub"
 				(path "/36dda7fd-e284-4ee0-b9cb-842fdde3c54e/842043d2-bca2-4e2b-b4fa-303380c6ca60"
-					(reference "R10")
+					(reference "R26")
 					(unit 1)
 				)
@@
 		(on_board yes)
 		(dnp no)
-		(property "Reference" "R5"
+		(property "Reference" "R21"
 			(at 96.266 76.454 0)
 			(effects
@@
 			(project "Multiport USB-C 2.0 hub"
 				(path "/36dda7fd-e284-4ee0-b9cb-842fdde3c54e/842043d2-bca2-4e2b-b4fa-303380c6ca60"
-					(reference "R5")
+					(reference "R21")
 					(unit 1)
 				)
@@
 		(on_board yes)
 		(dnp no)
-		(property "Reference" "R9"
+		(property "Reference" "R25"
 			(at 180.086 76.454 0)
 			(effects
@@
 			(project "Multiport USB-C 2.0 hub"
 				(path "/36dda7fd-e284-4ee0-b9cb-842fdde3c54e/842043d2-bca2-4e2b-b4fa-303380c6ca60"
-					(reference "R9")
+					(reference "R25")
 					(unit 1)
 				)
@@
 		(dnp no)
 		(fields_autoplaced yes)
-		(property "Reference" "#PWR07"
+		(property "Reference" "#PWR028"
 			(at 121.92 119.38 0)
 			(effects
@@
 			(project "Multiport USB-C 2.0 hub"
 				(path "/36dda7fd-e284-4ee0-b9cb-842fdde3c54e/842043d2-bca2-4e2b-b4fa-303380c6ca60"
-					(reference "#PWR07")
-					(unit 1)
-				)
+					(reference "#PWR028")
+					(unit 1)
+				)

Commit message: Update DFPs
Parts:
- added U10, U11, U12, U13, U8, U9: SRV05-4, Package_TO_SOT_SMD:SOT-23-6, symbol Power_Protection:SRV05-4
- DFP1, DFP2, DFP3, DFP4, DFP5, DFP6: value Downward facing port -> Downstream-facing port
Connections:
- net DFP1_D+: now also U8.3 (IO2)
- net DFP1_D-: now also U8.1 (IO1)
- net DFP2_D+: now also U9.3 (IO2)
- net DFP2_D-: now also U9.1 (IO1)
- net DFP3_D+: now also U10.3 (IO2)
- net DFP3_D-: now also U10.1 (IO1)
- net DFP4_D+: now also U11.3 (IO2)
- net DFP4_D-: now also U11.1 (IO1)
- net DFP5_D+: now also U12.3 (IO2)
- net DFP5_D-: now also U12.1 (IO1)
- net DFP6_D+: now also U13.3 (IO2)
- net DFP6_D-: now also U13.1 (IO1)
- net DFP_VBUS: now also U10.5 (VP), U11.5 (VP), U12.5 (VP), U13.5 (VP), U8.5 (VP), U9.5 (VP)
- net GND: now also U10.2 (VN), U11.2 (VN), U12.2 (VN), U13.2 (VN), U8.2 (VN), U9.2 (VN)
- net P5CC1: now reaches DFP5.A5 (CC1), R27.2
- net P5CC1: now also U12.4 (IO3)
- net P5CC2: now reaches DFP5.B5 (CC2), R28.2
- net P5CC2: now also U12.6 (IO4)
- net P1CC1: now reaches DFP1.A5 (CC1), R19.2
- net P1CC1: now also U8.4 (IO3)
- net P3CC2: now reaches DFP3.B5 (CC2), R24.2
- net P3CC2: now also U10.6 (IO4)
- net P4CC1: now reaches DFP4.A5 (CC1), R25.2
- net P4CC1: now also U11.4 (IO3)
- net P4CC2: now reaches DFP4.B5 (CC2), R26.2
- net P4CC2: now also U11.6 (IO4)
- net P2CC2: now reaches DFP2.B5 (CC2), R22.2
- net P2CC2: now also U9.6 (IO4)
- net P6CC1: now reaches DFP6.A5 (CC1), R29.2
- net P6CC1: now also U13.4 (IO3)
- net P6CC2: now reaches DFP6.B5 (CC2), R30.2
- net P6CC2: now also U13.6 (IO4)
- net P3CC1: now reaches DFP3.A5 (CC1), R23.2
- net P3CC1: now also U10.4 (IO3)
- net P1CC2: now reaches DFP1.B5 (CC2), R20.2
- net P1CC2: now also U8.6 (IO4)
- net P2CC1: now reaches DFP2.A5 (CC1), R21.2
- net P2CC1: now also U9.4 (IO3)
Other:
- moved on the sheet: DFP1, R19, R20

Commit message: footprints
Parts:
- R19, R20, R21, R22, R23, R24, R25, R26, R27, R28, R29, R30: footprint (none) -> Resistor_SMD:R_0603_1608Metric
- USBC3: renamed from DFP1; value Downstream-facing port -> DFP1
- USBC4: renamed from DFP2; value Downstream-facing port -> DFP2
- USBC5: renamed from DFP3; value Downstream-facing port -> DFP3
- USBC6: renamed from DFP4; value Downstream-facing port -> DFP4
- USBC7: renamed from DFP5; value Downstream-facing port -> DFP5
- USBC8: renamed from DFP6; value Downstream-facing port -> DFP6
Other:
- moved on the sheet: R25, R26, R27, R28, R29, R30, U11, U12, U13, USBC6, USBC7, USBC8
