File: Multiport USB-C 2.0 hub.kicad_sch (KiCad schematic)
At the start: 0 parts

Commit message: good first pass
Other:
- sheet Downward facing ports renamed Downstream-facing ports
- sheet Power delivery renamed Power management
- sheet Power management ports: added DFP_VBUS, PD_CC1, PD_CC2, PD_D+, PD_D-, PD_VBUS, UFP_VBUS; removed none
- sheet Upstream-facing ports ports: added PD_D+, PD_D-; removed none
- note added: "PD"
- note added: "Sink controller Power MUX Buck converter"
- note added: "x 6"
- note removed: "60W PD"
- company: (none) -> https://pips.engineering
- title: (none) -> Multiport USB-C 2.0 hub

Commit message: more work on USB hubs
Other:
- sheet USB hub ports: added DFP_VBUS; removed none
Changed lines of the file:
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@@
 		)
+	)
+	(junction
+		(at 181.61 104.14)
+		(diameter 0)
+		(color 0 0 0 0)
 	)
 	(wire
@@
 	(wire
 		(pts
+			(xy 181.61 85.09) (xy 184.15 85.09)
+		)
+		(stroke
+			(width 0)
+			(type default)
+		)
+	)
+	(wire
+		(pts
 			(xy 120.65 76.2) (xy 128.27 76.2)
 		)
@@
 		(pts
 			(xy 201.93 97.79) (xy 201.93 109.22)
+		)
+		(stroke
+			(width 0)
+			(type default)
+		)
+	)
+	(wire
+		(pts
+			(xy 181.61 104.14) (xy 181.61 85.09)
 		)
 		(stroke
@@
 			(effects
 				(font
+					(size 1.27 1.27)
+				)
+				(justify left)
+			)
+		)
+		(pin "DFP_VBUS" input
+			(at 184.15 85.09 180)
+			(effects
+				(font

Commit message: Update DFPs
Changed lines of the file:
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@@
 	)
 	(junction
-		(at 181.61 104.14)
+		(at 180.34 104.14)
 		(diameter 0)
 		(color 0 0 0 0)
@@
 	(wire
 		(pts
-			(xy 124.46 104.14) (xy 181.61 104.14)
+			(xy 124.46 104.14) (xy 180.34 104.14)
 		)
 		(stroke
@@
 	(wire
 		(pts
-			(xy 181.61 85.09) (xy 184.15 85.09)
+			(xy 180.34 85.09) (xy 184.15 85.09)
 		)
 		(stroke
@@
 	(wire
 		(pts
-			(xy 181.61 104.14) (xy 181.61 109.22)
+			(xy 180.34 104.14) (xy 180.34 109.22)
 		)
 		(stroke
@@
 	(wire
 		(pts
-			(xy 181.61 104.14) (xy 181.61 85.09)
+			(xy 180.34 104.14) (xy 180.34 85.09)
 		)
 		(stroke
@@
 	)
 	(sheet
-		(at 179.07 109.22)
-		(size 44.45 19.05)
+		(at 177.8 109.22)
+		(size 45.72 19.05)
 		(exclude_from_sim no)
 		(in_bom yes)
@@
 		)
 		(property "Sheetname" "Downstream-facing ports"
-			(at 178.816 130.556 0)
+			(at 177.546 130.556 0)
 			(effects
 				(font
@@
 		)
 		(property "Sheetfile" "DFPs.kicad_sch"
-			(at 179.07 131.318 0)
+			(at 177.8 131.318 0)
 			(effects
 				(font
@@
 		)
 		(pin "DFP_VBUS" bidirectional
-			(at 181.61 109.22 90)
-			(effects
-				(font
+			(at 180.34 109.22 90)
+			(effects
+				(font

Commit message: footprints
Changed lines of the file:
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@@
 			)
 		)
-		(pin "DFP_VBUS" bidirectional
+		(pin "DFP_VBUS" input
 			(at 180.34 109.22 90)
 			(effects
