File: PD.kicad_sch (KiCad schematic)
At the start: 0 parts

Commit message: good first pass
Parts:
- added C1: 1μF, symbol Device:C_Small
- added C2: Cbst, symbol Device:C_Small
- added C3: Cin, symbol Device:C_Small
- added C4: Css, symbol Device:C_Small
- added C5: Cout, symbol Device:C_Small
- added C6: 0.1μF, symbol Device:C_Small
- added D1: ~, symbol Device:D_Schottky_Small
- added L1: 3.3μH, symbol Device:L_Small
- added Q1: PMOS, symbol Simulation_SPICE:PMOS
- added R17, R18: ~, symbol Device:R_Small
- added R19: Rmc, symbol Device:R_Small
- added R20: Rfbt, symbol Device:R_Small
- added R21: Rfbb, symbol Device:R_Small
- added R22: Riset, symbol Device:R_Small
- added R23: 19kΩ, symbol Device:R_Small
- added R24: 30kΩ, symbol Device:R_Small
- added U3: HUSB238A-xxxxx-QN16R, Package_DFN_QFN:WQFN-16-1EP_3x3mm_P0.5mm_EP1.75x1.75mm, symbol Interface_USB:HUSB238A-xxxxx-QN16R
- added U4: TPS2121, Package_DFN_QFN:Texas_VQFN-HR-12_2x2.5mm_P0.5mm_ThermalVias, symbol TPS2121:TPS2121
- added U5: TPS56A37RPAR, TPS56A37:TPS56A37, symbol TPS56A37:TPS56A37RPAR
Connections:
- new net: C2.1, U5.7 (BOOT)
- new net: C2.2, L1.2, U5.6 (SW)
- new net: D1.2 (A), Q1.2 (G), R17.2, R18.1
- new net: R24.1, U4.10 (ILIM)
- new net: C6.1, U4.11 (SS)
- new net: C4.1, U5.5 (SS)
- new net: R20.2, R21.1, U5.2 (FB)
- new net: R22.1, U3.10 (SCL/SNK_ISET)
- new net: R23.1, U3.9 (SDA/SNK_VSET)
- new net: R19.1, U5.10 (MODE)
- new net DFP_VBUS: C5.1, L1.1, R20.1
- new net GATE: R18.2, U3.15 (GATE)
- new net GND: C1.2, C3.2, C4.2, C5.2, C6.2, R19.2, R21.2, R22.2, R23.2, R24.2, U3.12 (~{EN}), U3.17 (GND), U4.12 (GND), U4.3 (CP2), U4.4 (OV2), U4.5 (OV1), U4.6 (PR1), U5.3 (AGND), U5.9 (PGND)
- new net PD_CC1: U3.3 (CC1)
- new net PD_CC2: U3.4 (CC2)
- new net PD_D+: U3.1 (D+)
- new net PD_D-: U3.2 (D-)
- new net PD_SYS: Q1.1 (D), U4.7 (IN1)
- new net PD_VBUS: C1.1, D1.1 (K), Q1.3 (S), R17.1, U3.16 (VBUS)
- new net UFP_VBUS: U4.2 (IN2)
- new net VOUT: C3.1, U4.1 (OUT), U4.8 (OUT), U5.1 (EN), U5.8 (VIN)
- no-connect marks 0 -> 1
Other:
- note added: "20V"
- note added: "3.25A"
- note added: "6 USB ports Max 15W per port (5V x 3A) Total output 90W(5V x 3A x 6 ports) Sink max power 91W (28V x 3.25A)"
- note added: "IN1 = 5V - 20V IN2 = 5V"
- note added: "TODO: confirm ILIM value (3.25A) confirm priority confirm OVP"
- note added: "Vin = 5V - 20V Vout = 5V Iout = 10A"
- company: (none) -> https://pips.engineering
- title: (none) -> Power delivery components

Commit message: more work on USB hubs
Parts:
- R10: renamed from R19; value Rmc -> Rmd
- R7: renamed from R22; value Riset -> 21kΩ; now fitted
- renumbered C3 to C2, C2 to C3, C6 to C4, C4 to C6, R17 to R3, R18 to R4, R20 to R5, R23 to R6, R24 to R8, R21 to R9, U4 to U3, U5 to U4, U3 to U5
Other:
- note added: "3A"
- note added: "6 USB ports Max 7.5W per port (5V x 1.5A) Total output 45W(5V x 1.5A x 6 ports) Sink max power 60W (20V x 3A) Buck max power 50W (5V x 10A)"
- note added: "TODO: confirm ILIM value (≥3A) confirm priority confirm OVP"
- note removed: "3.25A"
- note removed: "6 USB ports Max 15W per port (5V x 3A) Total output 90W(5V x 3A x 6 ports) Sink max power 91W (28V x 3.25A)"
- note removed: "TODO: confirm ILIM value (3.25A) confirm priority confirm OVP"

Commit message: Update PD.kicad_sch
Other:
- note added: "TODO: Calculate resistor/cap values"
Changed lines of the file:
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@@
 		)
 	)
+	(text "TODO:\nCalculate resistor/cap values"
+		(exclude_from_sim no)
+		(at 241.808 85.598 0)
+		(effects
+			(font
+				(size 1.27 1.27)
+				(thickness 0.1588)
+			)
+		)
+	)
 	(text "IN1 = 5V - 20V\nIN2 = 5V"
 		(exclude_from_sim no)
@@
 					(font
 						(size 1.27 1.27)
+						(thickness 0.254)
+						(bold yes)
 					)
 					(justify left top)
@@
 					(font
 						(size 1.27 1.27)
+						(thickness 0.254)
+						(bold yes)
 					)
 					(justify left top)
@@
 			(table_cell "R_ISET kΩ"
 				(exclude_from_sim no)
-				(at 81.28 80.01 0)
+				(at 81.28 82.55 0)
 				(size 12.7 2.54)
 				(margins 0.9525 0.9525 0.9525 0.9525)
@@
 			(table_cell "Amperage"
 				(exclude_from_sim no)
-				(at 93.98 80.01 0)
+				(at 93.98 82.55 0)
 				(size 11.43 2.54)
 				(margins 0.9525 0.9525 0.9525 0.9525)
@@
 			(table_cell "21"
 				(exclude_from_sim no)
-				(at 81.28 82.55 0)
+				(at 81.28 85.09 0)
 				(size 12.7 2.54)
 				(margins 0.9525 0.9525 0.9525 0.9525)
@@
 					(font
 						(size 1.27 1.27)
+						(thickness 0.254)
+						(bold yes)
 					)
 					(justify left top)
@@
 			(table_cell "3A"
 				(exclude_from_sim no)
-				(at 93.98 82.55 0)
+				(at 93.98 85.09 0)
 				(size 11.43 2.54)
 				(margins 0.9525 0.9525 0.9525 0.9525)
@@
 					(font
 						(size 1.27 1.27)
+						(thickness 0.254)
+						(bold yes)
 					)
 					(justify left top)
@@
 			(table_cell "float"
 				(exclude_from_sim no)
-				(at 81.28 85.09 0)
+				(at 81.28 87.63 0)
 				(size 12.7 2.54)
 				(margins 0.9525 0.9525 0.9525 0.9525)
@@
 			(table_cell "3.25A"
 				(exclude_from_sim no)
-				(at 93.98 85.09 0)
+				(at 93.98 87.63 0)
 				(size 11.43 2.54)
 				(margins 0.9525 0.9525 0.9525 0.9525)

Commit message: footprints
Parts:
- added C3: 0.1μF, Capacitor_SMD:C_0603_1608Metric, symbol Device:C_Small
- added C7: 22μF, Capacitor_SMD:C_1206_3216Metric, symbol Device:C_Small
- C1: footprint (none) -> Capacitor_SMD:C_0603_1608Metric
- C2: value Cin -> 10μF; footprint (none) -> Capacitor_SMD:C_1206_3216Metric
- C4: renamed from C3; value Cbst -> 0.1μF; footprint (none) -> Capacitor_SMD:C_0603_1608Metric
- C5: renamed from C4; footprint (none) -> Capacitor_SMD:C_0603_1608Metric
- C6: renamed from C5; value Cout -> 22μF; footprint (none) -> Capacitor_SMD:C_1206_3216Metric
- C8: renamed from C6; value Css -> 47nF; footprint (none) -> Capacitor_SMD:C_0603_1608Metric
- R10: value Rmd -> 52.3kΩ; footprint (none) -> Resistor_SMD:R_0603_1608Metric
- R3, R4, R6, R7, R8: footprint (none) -> Resistor_SMD:R_0603_1608Metric
- R5: value Rfbt -> 73.2kΩ; footprint (none) -> Resistor_SMD:R_0603_1608Metric
- R9: value Rfbb -> 10kΩ; footprint (none) -> Resistor_SMD:R_0603_1608Metric
Connections:
- net DFP_VBUS: now also C7.1
- net GND: now also C3.2, C7.2
- net VOUT: now also C3.1
- no-connect marks 1 -> 7
Other:
- note removed: "TODO: Calculate resistor/cap values"
- moved on the sheet: C2, C4, C6, C8, L1, R10, R5, R6, R7, R9, U4
