File: UFP.kicad_sch (KiCad schematic)
At the start: 4 parts

Commit message: good first pass
Parts:
- added U6, U7: SRV05-4, Package_TO_SOT_SMD:SOT-23-6, symbol Power_Protection:SRV05-4
Connections:
- net GND: now also U6.2 (VN), U7.2 (VN)
- net PD_CC1: now also U6.1 (IO1)
- net PD_CC2: now also U6.3 (IO2)
- net PD_VBUS: now also U6.5 (VP)
- net UFP_D+: now also U7.6 (IO4)
- net UFP_D-: now also U7.4 (IO3)
- net UFP_VBUS: now also U7.5 (VP)
- net CC2: now reaches R2.1, UFP1.B5 (CC2)
- net CC2: now also U7.3 (IO2)
- net CC1: now reaches R1.2, UFP1.A5 (CC1)
- net CC1: now also U7.1 (IO1)
- net PD_D+: now reaches PD1.A6 (D+)
- net PD_D+: now also PD1.B6 (D+), U6.6 (IO4)
- net PD_D-: now reaches PD1.A7 (D-)
- net PD_D-: now also PD1.B7 (D-), U6.4 (IO3)
- no-connect marks 4 -> 0
Other:
- company: (none) -> https://pips.engineering
- title: (none) -> Upstream-facing ports
- moved on the sheet: PD1, R1, R2, UFP1

Commit message: more work on USB hubs
Parts:
- renumbered U6 to U1, U7 to U2
Changed lines of the file:
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@@
 		(dnp no)
 		(fields_autoplaced yes)
-		(property "Reference" "#PWR020"
+		(property "Reference" "#PWR02"
 			(at 179.07 104.14 0)
 			(effects
@@
 			(project "Multiport USB-C 2.0 hub"
 				(path "/36dda7fd-e284-4ee0-b9cb-842fdde3c54e/0d39d546-6b90-4921-ad72-df04e5c0c865"
-					(reference "#PWR020")
+					(reference "#PWR02")
 					(unit 1)
 				)
@@
 		(dnp no)
 		(fields_autoplaced yes)
-		(property "Reference" "U6"
+		(property "Reference" "U1"
 			(at 182.1881 69.85 0)
 			(effects
@@
 			(project "Multiport USB-C 2.0 hub"
 				(path "/36dda7fd-e284-4ee0-b9cb-842fdde3c54e/0d39d546-6b90-4921-ad72-df04e5c0c865"
-					(reference "U6")
+					(reference "U1")
 					(unit 1)
 				)
@@
 		(dnp no)
 		(fields_autoplaced yes)
-		(property "Reference" "#PWR01"
+		(property "Reference" "#PWR05"
 			(at 115.57 120.65 0)
 			(effects
@@
 			(project "Multiport USB-C 2.0 hub"
 				(path "/36dda7fd-e284-4ee0-b9cb-842fdde3c54e/0d39d546-6b90-4921-ad72-df04e5c0c865"
-					(reference "#PWR01")
+					(reference "#PWR05")
 					(unit 1)
 				)
@@
 		(dnp no)
 		(fields_autoplaced yes)
-		(property "Reference" "#PWR021"
+		(property "Reference" "#PWR01"
 			(at 144.78 90.17 0)
 			(effects
@@
 			(project "Multiport USB-C 2.0 hub"
 				(path "/36dda7fd-e284-4ee0-b9cb-842fdde3c54e/0d39d546-6b90-4921-ad72-df04e5c0c865"
-					(reference "#PWR021")
+					(reference "#PWR01")
 					(unit 1)
 				)
@@
 		(dnp no)
 		(fields_autoplaced yes)
-		(property "Reference" "#PWR02"
+		(property "Reference" "#PWR04"
 			(at 69.85 120.65 0)
 			(effects
@@
 			(project "Multiport USB-C 2.0 hub"
 				(path "/36dda7fd-e284-4ee0-b9cb-842fdde3c54e/0d39d546-6b90-4921-ad72-df04e5c0c865"
-					(reference "#PWR02")
+					(reference "#PWR04")
 					(unit 1)
 				)
@@
 		(dnp no)
 		(fields_autoplaced yes)
-		(property "Reference" "#PWR022"
+		(property "Reference" "#PWR03"
 			(at 223.52 104.14 0)
 			(effects
@@
 			(project "Multiport USB-C 2.0 hub"
 				(path "/36dda7fd-e284-4ee0-b9cb-842fdde3c54e/0d39d546-6b90-4921-ad72-df04e5c0c865"
-					(reference "#PWR022")
+					(reference "#PWR03")
 					(unit 1)
 				)
@@
 		(dnp no)
 		(fields_autoplaced yes)
-		(property "Reference" "U7"
+		(property "Reference" "U2"
 			(at 226.6381 69.85 0)
 			(effects
@@
 			(project "Multiport USB-C 2.0 hub"
 				(path "/36dda7fd-e284-4ee0-b9cb-842fdde3c54e/0d39d546-6b90-4921-ad72-df04e5c0c865"
-					(reference "U7")
-					(unit 1)
-				)
+					(reference "U2")
+					(unit 1)
+				)

Commit message: footprints
Parts:
- R1, R2: footprint (none) -> Resistor_SMD:R_0603_1608Metric
- USBC1: renamed from PD1; value PD port -> UFP1 - PD
- USBC2: renamed from UFP1; value Upstream-facing port -> UFP2 - data
Changed lines of the file:
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@@
 	(text_box "Upstream ports"
 		(exclude_from_sim no)
-		(at 57.15 62.23 0)
-		(size 91.44 60.96)
+		(at 54.61 62.23 0)
+		(size 93.98 60.96)
 		(margins 0.9525 0.9525 0.9525 0.9525)
 		(stroke
@@
 			)
 		)
-		(property "Footprint" ""
+		(property "Footprint" "Resistor_SMD:R_0603_1608Metric"
 			(at 139.7 83.82 0)
 			(effects
@@
 			)
 		)
-		(property "Footprint" ""
+		(property "Footprint" "Resistor_SMD:R_0603_1608Metric"
 			(at 139.7 81.28 0)
 			(effects
@@
 		(dnp no)
 		(fields_autoplaced yes)
-		(property "Reference" "PD1"
+		(property "Reference" "USBC1"
 			(at 69.85 68.58 0)
 			(effects
@@
 			)
 		)
-		(property "Value" "PD port"
+		(property "Value" "UFP1 - PD"
 			(at 69.85 71.12 0)
 			(effects
@@
 			(project "Multiport USB-C 2.0 hub"
 				(path "/36dda7fd-e284-4ee0-b9cb-842fdde3c54e/0d39d546-6b90-4921-ad72-df04e5c0c865"
-					(reference "PD1")
+					(reference "USBC1")
 					(unit 1)
 				)
@@
 		(dnp no)
 		(fields_autoplaced yes)
-		(property "Reference" "UFP1"
+		(property "Reference" "USBC2"
 			(at 115.57 68.58 0)
 			(effects
@@
 			)
 		)
-		(property "Value" "Upstream-facing port"
+		(property "Value" "UFP2 - data"
 			(at 115.57 71.12 0)
 			(effects
@@
 			(project "Multiport USB-C 2.0 hub"
 				(path "/36dda7fd-e284-4ee0-b9cb-842fdde3c54e/0d39d546-6b90-4921-ad72-df04e5c0c865"
-					(reference "UFP1")
+					(reference "USBC2")
 					(unit 1)
 				)
