File: USB hub IC.kicad_sch (KiCad schematic)
At the start: 4 parts, among them U1 FE1.1s, U2 FE1.1s

Commit message: good first pass
Connections:
- no-connect marks 0 -> 2
Other:
- company: (none) -> https://pips.engineering
- title: (none) -> USB 2.0 hub controllers + LEDs
- moved on the sheet: R15, R16, U1, U2

Commit message: more work on USB hubs
Parts:
- added C10, C7, C8, C9: 10μF, symbol Device:C_Small
- added D10: NC DFP7, symbol Device:LED_Small
- added D11: Hub2 A/S, symbol Device:LED_Small
- added D2: DFP1, symbol Device:LED_Small
- added D3: DFP4, symbol Device:LED_Small
- added D4: DFP2, symbol Device:LED_Small
- added D5: DFP5, symbol Device:LED_Small
- added D6: DFP3, symbol Device:LED_Small
- added D7: DFP6, symbol Device:LED_Small
- added D8: HUB2, symbol Device:LED_Small
- added D9: Hub1 A/S, symbol Device:LED_Small
- added R13, R14, R15, R16, R17, R18: ?Ω, symbol Device:R_Small
- added X1, X2: 12MHz, symbol Device:Crystal_Small
- U6: renamed from U1; value FE1.1s -> FE1.1s HUB1
- U7: renamed from U2; value FE1.1s -> FE1.1s HUB2
- renumbered R15 to R11, R16 to R12
Connections:
- net GND: now also C10.1, C7.1, C8.1, C9.1, R17.1, R18.1
- net at U7.12 (VD18_O): now also U7.28 (VD18), C10.2
- net at U7.13 (VD33): now also U7.21 (VD33_O), C9.2
- net DFP_VBUS: now reaches U7.18 (VBUSM)
- net DFP_VBUS: now also U6.18 (VBUSM), U6.20 (VDD5), U7.20 (VDD5)
- net at U7.2 (XOUT): now also X2.2
- net HUB2_DRV: now reaches U7.22 (DRV)
- net HUB2_DRV: now also D10.1 (K), D11.2 (A), D3.2 (A), D5.1 (K), D7.2 (A)
- net HUB2_LED1: now reaches U7.23 (LED1/EESCL)
- net HUB2_LED1: now also R14.1
- net HUB2_LED2: now reaches U7.24 (LED2)
- net HUB2_LED2: now also R16.1
- net at U7.3 (XIN): now also X2.1
- net at U6.12 (VD18_O): now also U6.28 (VD18), C8.2
- net at U6.13 (VD33): now also U6.21 (VD33_O), C7.2
- net at U6.2 (XOUT): now also X1.2
- net HUB1_DRV: now reaches U6.22 (DRV)
- net HUB1_DRV: now also D2.2 (A), D4.1 (K), D6.2 (A), D8.1 (K), D9.2 (A)
- net HUB1_LED1: now reaches U6.23 (LED1/EESCL)
- net HUB1_LED1: now also R13.1
- net HUB1_LED2: now reaches U6.24 (LED2)
- net HUB1_LED2: now also R15.1
- net at U6.3 (XIN): now also X1.1
- new net: D6.1 (K), D8.2 (A), R15.2
- new net: D2.1 (K), D4.2 (A), R13.2
- new net: D10.2 (A), D7.1 (K), R16.2
- new net: D3.1 (K), D5.2 (A), R14.2
- new net: D11.1 (K), R18.2
- new net: D9.1 (K), R17.2
Other:
- moved on the sheet: R11, R12, U6, U7

Commit message: footprints
Parts:
- C10: renamed from C8; footprint (none) -> Capacitor_SMD:C_1206_3216Metric
- C11: renamed from C9; footprint (none) -> Capacitor_SMD:C_1206_3216Metric
- C12: renamed from C10; footprint (none) -> Capacitor_SMD:C_1206_3216Metric
- C9: renamed from C7; footprint (none) -> Capacitor_SMD:C_1206_3216Metric
- D2, D3, D4, D5, D6, D7: footprint (none) -> LED_SMD:LED_0603_1608Metric
- R11: renamed from R13; footprint (none) -> Resistor_SMD:R_0603_1608Metric
- R12: renamed from R14; footprint (none) -> Resistor_SMD:R_0603_1608Metric
- R13: renamed from R15; footprint (none) -> Resistor_SMD:R_0603_1608Metric
- R14: renamed from R16; footprint (none) -> Resistor_SMD:R_0603_1608Metric
- R15: renamed from R17; footprint (none) -> Resistor_SMD:R_0603_1608Metric
- R16: renamed from R18; footprint (none) -> Resistor_SMD:R_0603_1608Metric
- R17: renamed from R11; footprint (none) -> Resistor_SMD:R_0603_1608Metric
- R18: renamed from R12; footprint (none) -> Resistor_SMD:R_0603_1608Metric
Changed lines of the file:
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@@
 			)
 		)
-		(property "Footprint" ""
+		(property "Footprint" "LED_SMD:LED_0603_1608Metric"
 			(at 182.88 58.42 90)
 			(effects
@@
 		(dnp no)
 		(fields_autoplaced yes)
-		(property "Reference" "R15"
+		(property "Reference" "R13"
 			(at 172.72 58.42 90)
 			(effects
@@
 			)
 		)
-		(property "Footprint" ""
+		(property "Footprint" "Resistor_SMD:R_0603_1608Metric"
 			(at 172.72 63.5 0)
 			(effects
@@
 			(project ""
 				(path "/36dda7fd-e284-4ee0-b9cb-842fdde3c54e/2aa657a2-7c4f-4981-901b-4c9e50c9501b"
-					(reference "R15")
+					(reference "R13")
 					(unit 1)
 				)
@@
 		(on_board yes)
 		(dnp no)
-		(property "Reference" "C9"
+		(property "Reference" "C11"
 			(at 120.65 33.274 0)
 			(effects
@@
 			)
 		)
-		(property "Footprint" ""
+		(property "Footprint" "Capacitor_SMD:C_1206_3216Metric"
 			(at 123.19 34.29 0)
 			(effects
@@
 			(project "Multiport USB-C 2.0 hub"
 				(path "/36dda7fd-e284-4ee0-b9cb-842fdde3c54e/2aa657a2-7c4f-4981-901b-4c9e50c9501b"
-					(reference "C9")
+					(reference "C11")
 					(unit 1)
 				)
@@
 		(dnp no)
 		(fields_autoplaced yes)
-		(property "Reference" "#PWR024"
+		(property "Reference" "#PWR022"
 			(at 203.2 74.93 0)
 			(effects
@@
 			(project ""
 				(path "/36dda7fd-e284-4ee0-b9cb-842fdde3c54e/2aa657a2-7c4f-4981-901b-4c9e50c9501b"
-					(reference "#PWR024")
+					(reference "#PWR022")
 					(unit 1)
 				)
@@
 		(dnp no)
 		(fields_autoplaced yes)
-		(property "Reference" "R13"
+		(property "Reference" "R11"
 			(at 172.72 38.1 90)
 			(effects
@@
 			)
 		)
-		(property "Footprint" ""
+		(property "Footprint" "Resistor_SMD:R_0603_1608Metric"
 			(at 172.72 43.18 0)
 			(effects
@@
 			(project ""
 				(path "/36dda7fd-e284-4ee0-b9cb-842fdde3c54e/2aa657a2-7c4f-4981-901b-4c9e50c9501b"
-					(reference "R13")
+					(reference "R11")
 					(unit 1)
 				)
@@
 		(dnp no)
 		(fields_autoplaced yes)
-		(property "Reference" "R16"
+		(property "Reference" "R14"
 			(at 223.52 58.42 90)
 			(effects
@@
 			)
 		)
-		(property "Footprint" ""
+		(property "Footprint" "Resistor_SMD:R_0603_1608Metric"
 			(at 223.52 63.5 0)
 			(effects
@@
 			(project "Multiport USB-C 2.0 hub"
 				(path "/36dda7fd-e284-4ee0-b9cb-842fdde3c54e/2aa657a2-7c4f-4981-901b-4c9e50c9501b"
-					(reference "R16")
+					(reference "R14")
 					(unit 1)
 				)
@@
 		(dnp no)
 		(fields_autoplaced yes)
-		(property "Reference" "#PWR022"
+		(property "Reference" "#PWR024"
 			(at 54.61 101.6 0)
 			(effects
@@
 			(project ""
 				(path "/36dda7fd-e284-4ee0-b9cb-842fdde3c54e/2aa657a2-7c4f-4981-901b-4c9e50c9501b"
-					(reference "#PWR022")
+					(reference "#PWR024")
 					(unit 1)
 				)
@@
 			)
 		)
-		(property "Footprint" ""
+		(property "Footprint" "LED_SMD:LED_0603_1608Metric"
 			(at 233.68 48.26 90)
 			(effects
@@
 		(dnp no)
 		(fields_autoplaced yes)
-		(property "Reference" "#PWR023"
+		(property "Reference" "#PWR025"
 			(at 120.65 101.6 0)
 			(effects
@@
 			(project "Multiport USB-C 2.0 hub"
 				(path "/36dda7fd-e284-4ee0-b9cb-842fdde3c54e/2aa657a2-7c4f-4981-901b-4c9e50c9501b"
-					(reference "#PWR023")
+					(reference "#PWR025")
 					(unit 1)
 				)
@@
 		(dnp no)
 		(fields_autoplaced yes)
-		(property "Reference" "#PWR025"
+		(property "Reference" "#PWR023"
 			(at 254 74.93 0)
 			(effects
@@
 			(project "Multiport USB-C 2.0 hub"
 				(path "/36dda7fd-e284-4ee0-b9cb-842fdde3c54e/2aa657a2-7c4f-4981-901b-4c9e50c9501b"
-					(reference "#PWR025")
+					(reference "#PWR023")
 					(unit 1)
 				)
@@
 		(dnp no)
 		(fields_autoplaced yes)
-		(property "Reference" "R17"
+		(property "Reference" "R15"
 			(at 200.66 63.5 90)
 			(effects
@@
 			)
 		)
-		(property "Footprint" ""
+		(property "Footprint" "Resistor_SMD:R_0603_1608Metric"
 			(at 200.66 68.58 0)
 			(effects
@@
 			(project "Multiport USB-C 2.0 hub"
 				(path "/36dda7fd-e284-4ee0-b9cb-842fdde3c54e/2aa657a2-7c4f-4981-901b-4c9e50c9501b"
-					(reference "R17")
+					(reference "R15")
 					(unit 1)
 				)
@@
 		(dnp no)
 		(fields_autoplaced yes)
-		(property "Reference" "R18"
+		(property "Reference" "R16"
 			(at 251.46 63.5 90)
 			(effects
@@
 			)
 		)
-		(property "Footprint" ""
+		(property "Footprint" "Resistor_SMD:R_0603_1608Metric"
 			(at 251.46 68.58 0)
 			(effects
@@
 			(project "Multiport USB-C 2.0 hub"
 				(path "/36dda7fd-e284-4ee0-b9cb-842fdde3c54e/2aa657a2-7c4f-4981-901b-4c9e50c9501b"
-					(reference "R18")
+					(reference "R16")
 					(unit 1)
 				)
@@
 			)
 		)
-		(property "Footprint" ""
+		(property "Footprint" "LED_SMD:LED_0603_1608Metric"
 			(at 182.88 48.26 90)
 			(effects
@@
 		(dnp no)
 		(fields_autoplaced yes)
-		(property "Reference" "C8"
+		(property "Reference" "C10"
 			(at 64.77 33.0262 0)
 			(effects
@@
 			)
 		)
-		(property "Footprint" ""
+		(property "Footprint" "Capacitor_SMD:C_1206_3216Metric"
 			(at 62.23 34.29 0)
 			(effects
@@
 			(project ""
 				(path "/36dda7fd-e284-4ee0-b9cb-842fdde3c54e/2aa657a2-7c4f-4981-901b-4c9e50c9501b"
-					(reference "C8")
+					(reference "C10")
 					(unit 1)
 				)
@@
 		)
 		(property "Description" "USB 2.0 High Speed 4-Port Hub Controller, SSOP-28"
+			(at 54.61 67.31 0)
+			(effects
+				(font
+					(size 1.27 1.27)
+				)
+				(hide yes)
+			)
+		)
+		(property "LCSC Part #" ""
 			(at 54.61 67.31 0)
 			(effects
@@
 		(dnp no)
 		(fields_autoplaced yes)
-		(property "Reference" "R11"
+		(property "Reference" "R17"
 			(at 34.29 91.4399 0)
 			(effects
@@
 			)
 		)
-		(property "Footprint" ""
+		(property "Footprint" "Resistor_SMD:R_0603_1608Metric"
 			(at 36.83 92.71 0)
 			(effects
@@
 			(project ""
 				(path "/36dda7fd-e284-4ee0-b9cb-842fdde3c54e/2aa657a2-7c4f-4981-901b-4c9e50c9501b"
-					(reference "R11")
+					(reference "R17")
 					(unit 1)
 				)
@@
 			)
 		)
-		(property "Footprint" ""
+		(property "Footprint" "LED_SMD:LED_0603_1608Metric"
 			(at 182.88 38.1 90)
 			(effects
@@
 		(dnp no)
 		(fields_autoplaced yes)
-		(property "Reference" "R14"
+		(property "Reference" "R12"
 			(at 223.52 38.1 90)
 			(effects
@@
 			)
 		)
-		(property "Footprint" ""
+		(property "Footprint" "Resistor_SMD:R_0603_1608Metric"
 			(at 223.52 43.18 0)
 			(effects
@@
 			(project "Multiport USB-C 2.0 hub"
 				(path "/36dda7fd-e284-4ee0-b9cb-842fdde3c54e/2aa657a2-7c4f-4981-901b-4c9e50c9501b"
-					(reference "R14")
+					(reference "R12")
 					(unit 1)
 				)
@@
 		(on_board yes)
 		(dnp no)
-		(property "Reference" "C7"
+		(property "Reference" "C9"
 			(at 54.61 33.274 0)
 			(effects
@@
 			)
 		)
-		(property "Footprint" ""
+		(property "Footprint" "Capacitor_SMD:C_1206_3216Metric"
 			(at 57.15 34.29 0)
 			(effects
@@
 			(project ""
 				(path "/36dda7fd-e284-4ee0-b9cb-842fdde3c54e/2aa657a2-7c4f-4981-901b-4c9e50c9501b"
-					(reference "C7")
+					(reference "C9")
 					(unit 1)
 				)
@@
 			)
 		)
-		(property "Footprint" ""
+		(property "Footprint" "LED_SMD:LED_0603_1608Metric"
 			(at 233.68 38.1 90)
 			(effects
@@
 		(dnp no)
 		(fields_autoplaced yes)
-		(property "Reference" "R12"
+		(property "Reference" "R18"
 			(at 100.33 91.4399 0)
 			(effects
@@
 			)
 		)
-		(property "Footprint" ""
+		(property "Footprint" "Resistor_SMD:R_0603_1608Metric"
 			(at 102.87 92.71 0)
 			(effects
@@
 			(project "Multiport USB-C 2.0 hub"
 				(path "/36dda7fd-e284-4ee0-b9cb-842fdde3c54e/2aa657a2-7c4f-4981-901b-4c9e50c9501b"
-					(reference "R12")
+					(reference "R18")
 					(unit 1)
 				)
@@
 			)
 		)
-		(property "Footprint" ""
+		(property "Footprint" "LED_SMD:LED_0603_1608Metric"
 			(at 233.68 58.42 90)
 			(effects
@@
 		(dnp no)
 		(fields_autoplaced yes)
-		(property "Reference" "C10"
+		(property "Reference" "C12"
 			(at 130.81 33.0262 0)
 			(effects
@@
 			)
 		)
-		(property "Footprint" ""
+		(property "Footprint" "Capacitor_SMD:C_1206_3216Metric"
 			(at 128.27 34.29 0)
 			(effects
@@
 			(project "Multiport USB-C 2.0 hub"
 				(path "/36dda7fd-e284-4ee0-b9cb-842fdde3c54e/2aa657a2-7c4f-4981-901b-4c9e50c9501b"
-					(reference "C10")
-					(unit 1)
-				)
+					(reference "C12")
+					(unit 1)
+				)
